Commit message: Upload robot data

File: Project2/catkin_ws/src/my_robot/urdf/my_robot.xacro (robot description, xacro)
@@ -1,4 +1,6 @@
 <?xml version='1.0'?>
 <robot name="my_robot" xmlns:xacro="http://www.ros.org/wiki/xacro">
+  <xacro:include filename="$(find my_robot)/urdf/my_robot.gazebo" />
+  <xacro:include filename="$(find my_robot)/urdf/materials.xacro" />
   <link name="robot_footprint"></link>
   <joint name="robot_footprint_joint" type="fixed">
@@ -83,4 +85,5 @@
         <box size=".4 .2 .1"/>
       </geometry>
+      <material name="blue"/>
     </visual>
     <collision name='back_caster_collision'>
@@ -130,5 +133,5 @@
       <origin xyz="0.0 0 0" rpy=" 0 1.5707 1.5707"/>
       <geometry>
-        <cylinder radius="0.099" length="0.048"/>
+        <cylinder radius="0.1" length="0.048"/>
       </geometry>
     </collision>
@@ -136,6 +139,7 @@
       <origin xyz="0.0 0 0" rpy=" 0 1.5707 1.5707"/>
       <geometry>
-        <cylinder radius="0.1" length="0.05"/>
+        <cylinder radius="0.11" length="0.05"/>
       </geometry>
+      <material name="green"/>
     </visual>
   </link>
@@ -161,5 +165,5 @@
       <origin xyz="0.0 0 0" rpy=" 0 1.5707 1.5707"/>
       <geometry>
-        <cylinder radius="0.099" length="0.048"/>
+        <cylinder radius="0.1" length="0.048"/>
       </geometry>
     </collision>
@@ -167,6 +171,7 @@
       <origin xyz="0.0 0 0" rpy=" 0 1.5707 1.5707"/>
       <geometry>
-        <cylinder radius="0.1" length="0.05"/>
+        <cylinder radius="0.11" length="0.05"/>
       </geometry>
+      <material name="green"/>
     </visual>
   </link>

Commit message: Modified the model file - I modified the wheel size following the guideline radius: 0.11->0.1 length: 0.48->0.5

File: Project2/catkin_ws/src/my_robot/urdf/my_robot.xacro (robot description, xacro)
@@ -133,5 +133,5 @@
       <origin xyz="0.0 0 0" rpy=" 0 1.5707 1.5707"/>
       <geometry>
-        <cylinder radius="0.1" length="0.048"/>
+        <cylinder radius="0.1" length="0.05"/>
       </geometry>
     </collision>
@@ -139,5 +139,5 @@
       <origin xyz="0.0 0 0" rpy=" 0 1.5707 1.5707"/>
       <geometry>
-        <cylinder radius="0.11" length="0.05"/>
+        <cylinder radius="0.1" length="0.05"/>
       </geometry>
       <material name="green"/>
@@ -165,5 +165,5 @@
       <origin xyz="0.0 0 0" rpy=" 0 1.5707 1.5707"/>
       <geometry>
-        <cylinder radius="0.1" length="0.048"/>
+        <cylinder radius="0.1" length="0.05"/>
       </geometry>
     </collision>
@@ -171,5 +171,5 @@
       <origin xyz="0.0 0 0" rpy=" 0 1.5707 1.5707"/>
       <geometry>
-        <cylinder radius="0.11" length="0.05"/>
+        <cylinder radius="0.1" length="0.05"/>
       </geometry>
       <material name="green"/>
